File: hardware/balanced-xlr/balanced-xlr.sch (KiCad schematic (older format))
At the start: 15 parts, among them J1 XLR3_Ground, J2 XLR3_Ground, J3 XLR3_Ground, J4 XLR3_Ground, SW1 SW_Push, SW2 SW_Push, U1 WeMos_D1_mini, U2 MCP4661

Commit message: balanced-xlr v1.0 layout
Parts:
- removed J1, J2: XLR3_Ground, symbol Connector:XLR3_Ground
- added C2: 220uF, Capacitor_THT:CP_Radial_D6.3mm_P2.50mm, symbol Device:CP
- added H1, H2, H3, H4: HOLE, homebrew:HOLE_5MM_#8, symbol Homebrew:HOLE
- added J1, J2: XLR3_Female, homebrew:NC3FAH, symbol Connector:XLR3
- C1: footprint (none) -> Capacitor_SMD:C_0603_1608Metric_Pad1.05x0.95mm_HandSolder; LCSC (none) -> C14663
- J3, J4: value XLR3_Ground -> XLR3_Ground_Male; footprint (none) -> homebrew:NC3MAH
- R1, R2: footprint (none) -> Resistor_SMD:R_0603_1608Metric_Pad1.05x0.95mm_HandSolder; LCSC (none) -> C23162
- R3, R4, R5, R6: value 2k2 -> 1k; footprint (none) -> Resistor_SMD:R_0603_1608Metric_Pad1.05x0.95mm_HandSolder; LCSC (none) -> C4190
- SW1, SW2: footprint (none) -> homebrew:SW_TACTILE_5.1MM_TS-1187A-C-D-B; LCSC (none) -> C318888
- U2: footprint (none) -> Package_SO:TSSOP-14_4.4x5mm_P0.65mm; LCSC (none) -> C145605
Connections:
- net +3V3: now also C2.1
- net GND: now also C2.2
- net IN_L_A: now also R5.1, J1.2; no longer R3.1
- net IN_L_B: now also R6.1, J1.3; no longer R4.2
- net IN_R_A: now also R3.1, J2.2; no longer R5.1
- net IN_R_B: now also R4.2, J2.3; no longer R6.1
- net OUT_L_A: now also R5.2, U2.7 (P1A); no longer R3.2, U2.8 (P0A)
- net OUT_L_B: now also R6.2, U2.6 (P1W); no longer R4.1, U2.9 (P0W)
- net OUT_R_A: now also R3.2, U2.8 (P0A); no longer R5.2, U2.7 (P1A)
- net OUT_R_B: now also R4.1, U2.9 (P0W); no longer R6.2, U2.6 (P1W)
- net SHIELD_L: now also J1.1
- net SHIELD_R: now also J2.1
- net CASE_L: no longer names the net of J3.G
- net CASE_R: no longer names the net of J4.G
- no-connect marks 16 -> 18
Changed lines of the file:
@@
 EESchema Schematic File Version 4
+LIBS:balanced-xlr-cache
 EELAYER 30 0
 EELAYER END
@@
 Text GLabel 1500 5250 3    50   Input ~ 0
 IN_R_B
-$Comp
-L Connector:XLR3_Ground J1
-U 1 1 5EA258AB
-P 1500 3700
-F 0 "J1" H 1500 4065 50  0000 C CNN
-F 1 "XLR3_Ground" H 1500 3974 50  0000 C CNN
-F 2 "" H 1500 3700 50  0001 C CNN
-F 3 " ~" H 1500 3700 50  0001 C CNN
-	1    1500 3700
-	1    0    0    -1
-$EndComp
-$Comp
-L Connector:XLR3_Ground J2
-U 1 1 5EA26903
-P 1500 4950
-F 0 "J2" H 1500 5315 50  0000 C CNN
-F 1 "XLR3_Ground" H 1500 5224 50  0000 C CNN
-F 2 "" H 1500 4950 50  0001 C CNN
-F 3 " ~" H 1500 4950 50  0001 C CNN
-	1    1500 4950
-	1    0    0    -1
-$EndComp
-Text GLabel 1400 4000 3    50   Input ~ 0
-CASE_L
-Text GLabel 1400 5250 3    50   Input ~ 0
-CASE_R
 Text Notes 900  3400 0    100  ~ 0
 IN
@@
 P 3550 3700
 F 0 "J3" H 3550 4065 50  0000 C CNN
-F 1 "XLR3_Ground" H 3550 3974 50  0000 C CNN
-F 2 "" H 3550 3700 50  0001 C CNN
+F 1 "XLR3_Ground_Male" H 3550 3974 50  0000 C CNN
+F 2 "homebrew:NC3MAH" H 3550 3700 50  0001 C CNN
 F 3 " ~" H 3550 3700 50  0001 C CNN
 	1    3550 3700
@@
 P 3550 4950
 F 0 "J4" H 3550 5315 50  0000 C CNN
-F 1 "XLR3_Ground" H 3550 5224 50  0000 C CNN
-F 2 "" H 3550 4950 50  0001 C CNN
+F 1 "XLR3_Ground_Male" H 3550 5224 50  0000 C CNN
+F 2 "homebrew:NC3MAH" H 3550 4950 50  0001 C CNN
 F 3 " ~" H 3550 4950 50  0001 C CNN
 	1    3550 4950
 	1    0    0    -1
 $EndComp
-Text GLabel 3450 4000 3    50   Input ~ 0
-CASE_L
-Text GLabel 3450 5250 3    50   Input ~ 0
-CASE_R
 Text Notes 2950 3400 0    100  ~ 0
 OUT
@@
 F 0 "U2" H 4650 1250 100 0000 C CNN
 F 1 "MCP4661" H 4450 2150 100 0000 C CNN
-F 2 "" H 4800 2300 100 0001 C CNN
+F 2 "Package_SO:TSSOP-14_4.4x5mm_P0.65mm" H 4800 2300 100 0001 C CNN
 F 3 "" H 4800 2300 100 0001 C CNN
+F 4 "C145605" H 4850 1700 50  0001 C CNN "LCSC"
 	1    4850 1700
 	1    0    0    -1
@@
 F 0 "R1" H 2470 1346 50  0000 L CNN
 F 1 "4k7" H 2470 1255 50  0000 L CNN
-F 2 "" V 2330 1300 50  0001 C CNN
+F 2 "Resistor_SMD:R_0603_1608Metric_Pad1.05x0.95mm_HandSolder" V 2330 1300 50  0001 C CNN
 F 3 "~" H 2400 1300 50  0001 C CNN
+F 4 "C23162" H 2400 1300 50  0001 C CNN "LCSC"
 	1    2400 1300
 	1    0    0    -1
@@
 F 0 "R2" H 2920 1446 50  0000 L CNN
 F 1 "4k7" H 2920 1355 50  0000 L CNN
-F 2 "" V 2780 1400 50  0001 C CNN
+F 2 "Resistor_SMD:R_0603_1608Metric_Pad1.05x0.95mm_HandSolder" V 2780 1400 50  0001 C CNN
 F 3 "~" H 2850 1400 50  0001 C CNN
+F 4 "C23162" H 2850 1400 50  0001 C CNN "LCSC"
 	1    2850 1400
 	1    0    0    -1
@@
 F 0 "C1" H 5165 996 50  0000 L CNN
 F 1 "0.1uF" H 5165 905 50  0000 L CNN
-F 2 "" H 5088 800 50  0001 C CNN
+F 2 "Capacitor_SMD:C_0603_1608Metric_Pad1.05x0.95mm_HandSolder" H 5088 800 50  0001 C CNN
 F 3 "~" H 5050 950 50  0001 C CNN
+F 4 "C14663" H 5050 950 50  0001 C CNN "LCSC"
 	1    5050 950
 	1    0    0    -1
@@
 NoConn ~ 4250 2050
 Text GLabel 5950 1500 2    50   Input ~ 0
-IN_L_A
+IN_R_A
 $Comp
 L Device:R R3
@@
 P 5800 1500
 F 0 "R3" V 5800 1500 50  0000 C CNN
-F 1 "2k2" V 5684 1500 50  0000 C CNN
-F 2 "" V 5730 1500 50  0001 C CNN
+F 1 "1k" V 5684 1500 50  0000 C CNN
+F 2 "Resistor_SMD:R_0603_1608Metric_Pad1.05x0.95mm_HandSolder" V 5730 1500 50  0001 C CNN
 F 3 "~" H 5800 1500 50  0001 C CNN
+F 4 "C4190" V 5800 1500 50  0001 C CNN "LCSC"
 	1    5800 1500
 	0    1    1    0
@@
 P 5800 1600
 F 0 "R4" V 5800 1600 50  0000 C CNN
-F 1 "2k2" V 5900 1600 50  0000 C CNN
-F 2 "" V 5730 1600 50  0001 C CNN
+F 1 "1k" V 5900 1600 50  0000 C CNN
+F 2 "Resistor_SMD:R_0603_1608Metric_Pad1.05x0.95mm_HandSolder" V 5730 1600 50  0001 C CNN
 F 3 "~" H 5800 1600 50  0001 C CNN
+F 4 "C4190" V 5800 1600 50  0001 C CNN "LCSC"
 	1    5800 1600
 	0    -1   1    0
 $EndComp
 Text GLabel 5950 1600 2    50   Input ~ 0
-IN_L_B
+IN_R_B
 Text GLabel 5650 1250 2    50   Input ~ 0
-OUT_L_A
+OUT_R_A
 Text GLabel 5650 1800 2    50   Input ~ 0
-OUT_L_B
+OUT_R_B
 $Comp
 L Device:R R5
@@
 P 6550 1850
 F 0 "R5" V 6550 1850 50  0000 C CNN
-F 1 "2k2" V 6434 1850 50  0000 C CNN
-F 2 "" V 6480 1850 50  0001 C CNN
+F 1 "1k" V 6434 1850 50  0000 C CNN
+F 2 "Resistor_SMD:R_0603_1608Metric_Pad1.05x0.95mm_HandSolder" V 6480 1850 50  0001 C CNN
 F 3 "~" H 6550 1850 50  0001 C CNN
+F 4 "C4190" V 6550 1850 50  0001 C CNN "LCSC"
 	1    6550 1850
 	0    1    1    0
@@
 P 6550 1950
 F 0 "R6" V 6550 1950 50  0000 C CNN
-F 1 "2k2" V 6650 1950 50  0000 C CNN
-F 2 "" V 6480 1950 50  0001 C CNN
+F 1 "1k" V 6650 1950 50  0000 C CNN
+F 2 "Resistor_SMD:R_0603_1608Metric_Pad1.05x0.95mm_HandSolder" V 6480 1950 50  0001 C CNN
 F 3 "~" H 6550 1950 50  0001 C CNN
+F 4 "C4190" V 6550 1950 50  0001 C CNN "LCSC"
 	1    6550 1950
 	0    1    1    0
@@
 	6400 1850 6350 1850
 Text GLabel 6700 1850 2    50   Input ~ 0
-IN_R_A
+IN_L_A
 Text GLabel 6700 1950 2    50   Input ~ 0
-IN_R_B
+IN_L_B
 Text GLabel 6400 1600 2    50   Input ~ 0
-OUT_R_A
+OUT_L_A
 Text GLabel 6400 2150 2    50   Input ~ 0
-OUT_R_B
+OUT_L_B
 Wire Wire Line
 	6400 1950 6350 1950
@@
 F 0 "SW1" H 2550 2235 50  0000 C CNN
 F 1 "SW_Push" H 2550 2144 50  0000 C CNN
-F 2 "" H 2550 2150 50  0001 C CNN
+F 2 "homebrew:SW_TACTILE_5.1MM_TS-1187A-C-D-B" H 2550 2150 50  0001 C CNN
 F 3 "~" H 2550 2150 50  0001 C CNN
+F 4 "C318888" H 2550 1950 50  0001 C CNN "LCSC"
 	1    2550 1950
 	1    0    0    -1
@@
 F 0 "SW2" H 2550 2250 50  0000 C CNN
 F 1 "SW_Push" H 2550 2350 50  0000 C CNN
-F 2 "" H 2550 2250 50  0001 C CNN
+F 2 "homebrew:SW_TACTILE_5.1MM_TS-1187A-C-D-B" H 2550 2250 50  0001 C CNN
 F 3 "~" H 2550 2250 50  0001 C CNN
+F 4 "C318888" H 2550 2050 50  0001 C CNN "LCSC"
 	1    2550 2050
 	-1   0    0    1
@@
 $EndComp
 Connection ~ 1900 2550
+$Comp
+L Connector:XLR3 J1
+U 1 1 5EA3D1AD
+P 1500 3700
+F 0 "J1" H 1500 4065 50  0000 C CNN
+F 1 "XLR3_Female" H 1500 3974 50  0000 C CNN
+F 2 "homebrew:NC3FAH" H 1500 3700 50  0001 C CNN
+F 3 " ~" H 1500 3700 50  0001 C CNN
+	1    1500 3700
+	1    0    0    -1
+$EndComp
+$Comp
+L Connector:XLR3 J2
+U 1 1 5EA3FC49
+P 1500 4950
+F 0 "J2" H 1500 5315 50  0000 C CNN
+F 1 "XLR3_Female" H 1500 5224 50  0000 C CNN
+F 2 "homebrew:NC3FAH" H 1500 4950 50  0001 C CNN
+F 3 " ~" H 1500 4950 50  0001 C CNN
+	1    1500 4950
+	1    0    0    -1
+$EndComp
+NoConn ~ 3450 4000
+NoConn ~ 3450 5250
+$Comp
+L Homebrew:HOLE H1
+U 1 1 5EA4B2BA
+P 4900 3200
+F 0 "H1" H 5009 3253 60  0000 L CNN
+F 1 "HOLE" H 5009 3147 60  0000 L CNN
+F 2 "homebrew:HOLE_5MM_#8" H 4900 3200 60  0001 C CNN
+F 3 "" H 4900 3200 60  0001 C CNN
+	1    4900 3200
+	1    0    0    -1
+$EndComp
+$Comp
+L Homebrew:HOLE H2
+U 1 1 5EA4B774
+P 4900 3400
+F 0 "H2" H 5009 3453 60  0000 L CNN
+F 1 "HOLE" H 5009 3347 60  0000 L CNN
+F 2 "homebrew:HOLE_5MM_#8" H 4900 3400 60  0001 C CNN
+F 3 "" H 4900 3400 60  0001 C CNN
+	1    4900 3400
+	1    0    0    -1
+$EndComp
+$Comp
+L Homebrew:HOLE H3
+U 1 1 5EA4BA33
+P 4900 3600
+F 0 "H3" H 5009 3653 60  0000 L CNN
+F 1 "HOLE" H 5009 3547 60  0000 L CNN
+F 2 "homebrew:HOLE_5MM_#8" H 4900 3600 60  0001 C CNN
+F 3 "" H 4900 3600 60  0001 C CNN
+	1    4900 3600
+	1    0    0    -1
+$EndComp
+$Comp
+L Homebrew:HOLE H4
+U 1 1 5EA4BDAA
+P 4900 3800
+F 0 "H4" H 5009 3853 60  0000 L CNN
+F 1 "HOLE" H 5009 3747 60  0000 L CNN
+F 2 "homebrew:HOLE_5MM_#8" H 4900 3800 60  0001 C CNN
+F 3 "" H 4900 3800 60  0001 C CNN
+	1    4900 3800
+	1    0    0    -1
+$EndComp
+$Comp
+L Device:CP C2
+U 1 1 5EA5F14E
+P 5500 950
+F 0 "C2" H 5618 996 50  0000 L CNN
+F 1 "220uF" H 5618 905 50  0000 L CNN
+F 2 "Capacitor_THT:CP_Radial_D6.3mm_P2.50mm" H 5538 800 50  0001 C CNN
+F 3 "~" H 5500 950 50  0001 C CNN
+	1    5500 950
+	1    0    0    -1
+$EndComp
+Wire Wire Line
+	5050 800  5500 800
+Connection ~ 5050 800
+Wire Wire Line
+	5500 1100 5050 1100
+Connection ~ 5050 1100
 $EndSCHEMATC
